Commit message: extended code for right arm: adapt urdf file, ik

File: c++/src/urdf/yumi_right.urdf (robot description, URDF)
Before this commit: robot yumi, 9 links, 8 joints
Joints:
- joint yumi_joint_6_r: origin xyz=0.0283 0.0372 -0.0005 rpy=-1.57079632679 0.0 0.0 -> xyz=0.0273 0.1165 -0.0007 rpy=1.57079632679 0.0 3.14159
