Commit message: forward kinematics for both arms

File: c++/src/urdf/yumi_left.urdf (robot description, URDF)
Before this commit: robot yumi, 23 links, 22 joints
Links:
- removed link gripper_l_base
- removed link gripper_l_finger_l
- removed link gripper_l_finger_r
- removed link gripper_r_base
- removed link gripper_r_finger_l
- removed link gripper_r_finger_r
- removed link world
- removed link yumi_link_1_r
- removed link yumi_link_2_r
- removed link yumi_link_3_r
- removed link yumi_link_4_r
- removed link yumi_link_5_r
- removed link yumi_link_6_r
- removed link yumi_link_7_r
- link yumi_body: geometry 
- link yumi_link_1_l: geometry 
- link yumi_link_2_l: geometry 
- link yumi_link_3_l: geometry 
- link yumi_link_4_l: geometry 
- link yumi_link_5_l: geometry 
- link yumi_link_6_l: geometry 
- link yumi_link_7_l: geometry 
Joints:
- removed joint gripper_l_joint
- removed joint gripper_l_joint_m
- removed joint gripper_r_joint
- removed joint gripper_r_joint_m
- removed joint world_joint
- removed joint yumi_joint_1_r
- removed joint yumi_joint_2_r
- removed joint yumi_joint_3_r
- removed joint yumi_joint_4_r
- removed joint yumi_joint_5_r
- removed joint yumi_joint_6_r
- removed joint yumi_joint_7_r
- removed joint yumi_link_7_l_joint
- removed joint yumi_link_7_r_joint

Commit message: modified urdf files to match end effector in robot studio and updating cad files

File: c++/src/urdf/yumi_left.urdf (robot description, URDF)
Before this commit: robot yumi, 9 links, 8 joints
Joints:
- joint yumi_joint_6_l: origin xyz=0.027 0.029 0.0 rpy=-1.57079632679 0.0 0.0 -> xyz=0.0283 0.0575 -0.0005 rpy=-1.57079632679 0.0 0.0

File: c++/src/urdf/yumi_right.urdf (robot description, URDF)
Before this commit: robot yumi, 9 links, 8 joints
Joints:
- joint yumi_joint_6_r: origin xyz=0.027 0.029 0.0 rpy=-1.57079632679 0.0 0.0 -> xyz=0.0283 0.0372 -0.0005 rpy=-1.57079632679 0.0 0.0

Commit message: everything works now, but there is a bug in genpaths.py

File: c++/src/urdf/yumi_left.urdf (robot description, URDF)
Before this commit: robot yumi, 9 links, 8 joints
Joints:
- joint yumi_joint_6_l: axis 0 0 1 -> 1 0 0; origin xyz=0.0283 0.0575 -0.0005 rpy=-1.57079632679 0.0 0.0 -> xyz=0.0283 0.0575 -0.0005 rpy=0.0 0.0 1.57079632679

File: c++/src/urdf/yumi_right.urdf (robot description, URDF)
Before this commit: robot yumi, 9 links, 8 joints
Joints:
- joint yumi_joint_6_r: axis 0 0 1 -> 1 0 0; origin xyz=0.0273 0.1165 -0.0007 rpy=1.57079632679 0.0 3.14159 -> xyz=0.0273 0.1165 -0.0007 rpy=0.0 0.0 1.57079632679
