Commit message: force control plots v1

File: c++/models/urdf/yumi_left.urdf (robot description, URDF)
Before this commit: robot yumi, 9 links, 8 joints
Joints:
- joint yumi_joint_6_l: origin xyz=0.0283 0.0575 -0.0005 rpy=0.0 0.0 1.57079632679 -> xyz=0.02716 0.056592 -0.001031 rpy=0.0 0.0 1.57079632679

File: c++/models/urdf/yumi_left_original.urdf (robot description, URDF)
Before this commit: robot yumi, 9 links, 8 joints
Links:
- removed link yumi_link_1_r
- removed link yumi_link_2_r
- removed link yumi_link_3_r
- removed link yumi_link_4_r
- removed link yumi_link_5_r
- removed link yumi_link_6_r
- removed link yumi_link_7_r
- added link yumi_link_1_l, mass 2
- added link yumi_link_2_l, mass 2
- added link yumi_link_3_l, mass 2
- added link yumi_link_4_l, mass 2
- added link yumi_link_5_l, mass 2
- added link yumi_link_6_l, mass 2
- added link yumi_link_7_l, mass 2
Joints:
- removed joint yumi_joint_1_r
- removed joint yumi_joint_2_r
- removed joint yumi_joint_3_r
- removed joint yumi_joint_4_r
- removed joint yumi_joint_5_r
- removed joint yumi_joint_6_r
- removed joint yumi_joint_7_r
- added joint yumi_joint_1_l: type revolute, parent yumi_body, child yumi_link_1_l, origin xyz=0.05355 0.07250 0.41492 rpy=0.9781 -0.5716 2.3180, axis 0 0 1, limit lower=-2.94087978961 upper=2.94087978961 effort=300 velocity=3.14159265359
- added joint yumi_joint_2_l: type revolute, parent yumi_link_1_l, child yumi_link_2_l, origin xyz=0.03 0.0 0.1 rpy=1.57079632679 0.0 0.0, axis 0 0 1, limit lower=-2.50454747661 upper=0.759218224618 effort=300 velocity=3.14159265359
- added joint yumi_joint_3_l: type revolute, parent yumi_link_3_l, child yumi_link_4_l, origin xyz=-0.04188 0.0 0.07873 rpy=1.57079632679 -1.57079632679 0.0, axis 0 0 1, limit lower=-2.15548162621 upper=1.3962634016 effort=300 velocity=3.14159265359
- added joint yumi_joint_4_l: type revolute, parent yumi_link_4_l, child yumi_link_5_l, origin xyz=0.0405 0.16461 0.0 rpy=-1.57079632679 0.0 0.0, axis 0 0 1, limit lower=-5.06145483078 upper=5.06145483078 effort=300 velocity=6.98131700798
- added joint yumi_joint_5_l: type revolute, parent yumi_link_5_l, child yumi_link_6_l, origin xyz=-0.027 0 0.10039 rpy=1.57079632679 0.0 0.0, axis 0 0 1, limit lower=-1.53588974176 upper=2.40855436775 effort=300 velocity=6.98131700798
- added joint yumi_joint_6_l: type revolute, parent yumi_link_6_l, child yumi_link_7_l, origin xyz=0.027 0.029 0.0 rpy=0.0 0.0 0.0, axis 1 0 0, limit lower=-3.99680398707 upper=3.99680398707 effort=300 velocity=6.98131700798
- added joint yumi_joint_7_l: type revolute, parent yumi_link_2_l, child yumi_link_3_l, origin xyz=-0.03 0.17283 0.0 rpy=-1.57079632679 0.0 0.0, axis 0 0 1, limit lower=-2.94087978961 upper=2.94087978961 effort=300 velocity=3.14159265359

File: c++/models/urdf/yumi_right_original.urdf (robot description, URDF)
Before this commit: robot yumi, 9 links, 8 joints
Joints:
- joint yumi_joint_6_r: axis 1 0 0 -> 0 0 1; origin xyz=0.027101 0.116653 -0.00047 rpy=0.0 0.0 1.57079632679 -> xyz=0.027 0.029 0.0 rpy=-1.57079632679 0.0 0.0
